Commit message: update finding meshes

File: zed_wrapper/urdf/zed_macro.urdf.xacro (robot description, xacro)
@@ -114,5 +114,5 @@
           <origin xyz="${screw_offset_x} 0 ${screw_offset_z}" rpy="0 0 0"/>
           <geometry>
-<mesh filename="package://zed_msgs/meshes/${model}.stl" />
+<mesh filename="$(find zed_msgs)/meshes/${model}.stl" />
           </geometry>
           <material name="${model}_mat" />
@@ -121,5 +121,5 @@
           <origin xyz="${screw_offset_x} 0 ${screw_offset_z}" rpy="0 0 0"/>
           <geometry>
-<mesh filename="package://zed_msgs/meshes/${model}.stl" />
+<mesh filename="$(find zed_msgs)/meshes/${model}.stl" />
           </geometry>
         </collision>
@@ -138,5 +138,5 @@
             <origin xyz="0 0 0" rpy="0 0 0"/>
             <geometry>
-  <mesh filename="package://zed_msgs/meshes/${model}.stl" />
+  <mesh filename="$(find zed_msgs)/meshes/${model}.stl" />
             </geometry>
             <material name="${model}_mat" />
@@ -145,5 +145,5 @@
             <origin xyz="0 0 0" rpy="0 0 0"/>
             <geometry>
-  <mesh filename="package://zed_msgs/meshes/${model}.stl" />
+  <mesh filename="$(find zed_msgs)/meshes/${model}.stl" />
             </geometry>
           </collision>
@@ -167,5 +167,5 @@
             <origin xyz="0 0 0" rpy="0 0 0"/>
             <geometry>
-  <mesh filename="package://zed_msgs/meshes/${model}.stl" />
+  <mesh filename="$(find zed_msgs)/meshes/${model}.stl" />
             </geometry>
             <material name="${model}_mat" />
@@ -174,5 +174,5 @@
             <origin xyz="0 0 0" rpy="0 0 0"/>
             <geometry>
-  <mesh filename="package://zed_msgs/meshes/${model}.stl" />
+  <mesh filename="$(find zed_msgs)/meshes/${model}.stl" />
             </geometry>
           </collision>
